Commit message: added collision

File: src/my_robot_description/urdf/my_robot.urdf.xacro (robot description, xacro)
@@ -1,79 +1,5 @@
 <?xml version="1.0"?>
 <robot name="my_robot" xmlns:xacro="http://www.ros.org/wiki/xacro">
-    <xacro:property name="base_lenght" value="2"/>
-    <xacro:property name="base_width" value="0.4"/>
-    <xacro:property name="base_height" value="0.2"/>
-    <xacro:property name="wheel_radius" value="0.1"/>
-    <xacro:property name="wheel_lenght" value="0.05"/>
-    <material name="yellowish">
-        <color rgba="1 0.7 0 0.8"/>
-    </material>
-    <material name="second">
-        <color rgba="0.3 0.3 0.25 1"/>
-    </material>
-    <material name="third">
-    <color rgba="0.8 0.3 0 1"/>
-    </material>
-    <link name="base_link">
-        <visual>
-            <geometry>
-                <box size="${base_lenght} ${base_width} ${base_height}" />
-            </geometry>
-            <origin xyz="0 0 ${base_height/2.0}" rpy="0 0 0"/>
-            <material name="yellowish"/>
-        </visual>
-    </link>
-    <link name ="right_wheel_link">
-        <visual>
-            <geometry>
-                <cylinder  radius = "${wheel_radius}" length="${wheel_lenght}"/>
-            </geometry>
-            <origin xyz="0 0 0" rpy="${pi/2.0} 0 0"/>
-            <material name="second"/>
-        </visual>
-    </link>
-    <link name ="left_wheel_link">
-        <visual>
-            <geometry>
-                <cylinder  radius = "${wheel_radius}" length="${wheel_lenght}"/>
-            </geometry>
-            <origin xyz="0 0 0" rpy="${pi/2.0} 0 0"/>
-            <material name="second"/>
-        </visual>
-    </link>
-    <link name="base_footprint">
-        <visual>
-        </visual>
-    </link>
-    <link name ="caster_wheel_link">
-        <visual>
-            <geometry>
-                <sphere radius = "${wheel_radius/2.0}"/>
-            </geometry>
-            <origin xyz="0 0 0" rpy="0 0 0"/>
-            <material name="second"/>
-        </visual>
-    </link>
-    <joint name="base_right_wheel_joint" type="continuous">
-        <parent link="base_link"/>
-        <child link="right_wheel_link"/>
-        <origin xyz="${-base_lenght/4.0} ${-(base_width + wheel_lenght)/2.0} 0" rpy="0 0 0"/>
-        <axis xyz = "0 1 0"/>
-    </joint>
-    <joint name="base_left_wheel_joint" type="continuous">
-        <parent link="base_link"/>
-        <child link="left_wheel_link"/>
-        <origin xyz="${-base_lenght/4.0} ${(base_width + wheel_lenght)/2.0} 0" rpy="0 0 0"/>
-        <axis xyz = "0 1 0"/>
-    </joint>
-    <joint name="base_caster_wheel_joint" type="fixed">
-        <parent link="base_link"/>
-        <child link="caster_wheel_link"/>
-        <origin xyz="${base_lenght/ 3.0} 0 ${-wheel_radius / 2.0}" rpy="0 0 0"/>
-    </joint>
-    <joint name="base_joint" type ="fixed">
-            <parent link ="base_footprint"/>
-            <child link ="base_link"/>
-            <origin xyz="0 0 ${wheel_radius}" rpy = "0 0 0 "/>
-    </joint>
+    <xacro:include filename="common_properties.urdf.xacro"/>
+    <xacro:include filename="mobile_base.urdf.xacro"/>
 </robot>
