Commit message: added my_robot_bringup

File: src/my_robot_description/urdf/mobile_base.urdf.xacro (robot description, xacro)
@@ -74,5 +74,5 @@
         <parent link="base_link"/>
         <child link="left_wheel_link"/>
-        <origin xyz="${-base_lenght/4.0} ${(base_width +wheel_height)/2.0} 0" rpy="0 0 0"/>
+        <origin xyz="${-base_lenght/4.0} ${(base_width + wheel_height)/2.0} 0" rpy="0 0 0"/>
         <axis xyz = "0 1 0"/>
     </joint>
